File: PCB/LoraTimerSender/LoraTimerSender.kicad_pcb (KiCad board)
At the start: 2 copper layers, 31.2 x 26 mm, 8 parts, among them J1 BC501SM-TR, U2 DS3231MZ

Commit message: added all working codes separately
Parts:
- moved U1 0.10 mm to (129.2, 89.3)
Routing:
- net GND: track 15.0 -> 73.9 mm, vias 1 -> 2
- net VDD: track 17.7 -> 47.7 mm
- removed copper zone on B.Cu, net GND
- removed copper zone on F.Cu, net GND
Other:
- board size 31.2 x 26 mm -> 50.2 x 25.8 mm
